File: motor_driver/motor_driver.kicad_pcb (KiCad board)
At the start: 2 copper layers, 41 parts, among them J1 Power_in, J2 Conn_01x09, J3 Conn_01x10, J4 Screw_Terminal_01x03, Q1 N_MOSFET, Q10 N_MOSFET, Q11 N_MOSFET, Q12 N_MOSFET, Q2 N_MOSFET, Q3 N_MOSFET, Q4 N_MOSFET, Q5 N_MOSFET, Q6 N_MOSFET, Q7 N_MOSFET, Q8 N_MOSFET, Q9 N_MOSFET, U1 DRV8303

Commit message: Finished layout and generated gerbers
Parts:
- removed J3: Conn_01x10, Pin_Headers:Pin_Header_Straight_1x10_Pitch2.54mm
- added C14: CP1, Capacitors_SMD:CP_Elec_6.3x7.7, F.Cu at (168.4, 113.3)
- added D1: LED, LEDs:LED_0805, F.Cu at (205.5, 109.5)
- added R12: 1KR, Resistors_SMD:R_0805, F.Cu at (205.5, 105.5)
- added REF**: MountingHole_3.2mm_M3, Mounting_Holes:MountingHole_3.2mm_M3, F.Cu at (212.0, 99.0)
- added REF**: stitch_via, my_SMD:stitch_via0.2mm, F.Cu at (203.0, 112.0)
- added REF**: stitch_via, my_SMD:stitch_via0.2mm, F.Cu at (193.5, 133.8)
- added REF**: stitch_via, my_SMD:stitch_via0.2mm, F.Cu at (193.5, 134.2)
- added REF**: stitch_via, my_SMD:stitch_via0.2mm, F.Cu at (194.5, 134.2)
- added REF**: stitch_via, my_SMD:stitch_via0.2mm, F.Cu at (195.0, 133.8)
- added REF**: stitch_via, my_SMD:stitch_via0.2mm, F.Cu at (194.5, 133.8)
- added REF**: stitch_via, my_SMD:stitch_via0.2mm, F.Cu at (195.5, 133.8)
- added REF**: stitch_via, my_SMD:stitch_via0.2mm, F.Cu at (196.0, 133.8)
- added REF**: stitch_via, my_SMD:stitch_via0.2mm, F.Cu at (195.0, 134.2)
- added REF**: stitch_via, my_SMD:stitch_via0.2mm, F.Cu at (195.5, 134.2)
- added REF**: stitch_via, my_SMD:stitch_via0.2mm, F.Cu at (196.0, 134.2)
- added REF**: stitch_via, my_SMD:stitch_via0.2mm, F.Cu at (203.0, 108.0)
- added REF**: stitch_via, my_SMD:stitch_via0.2mm, F.Cu at (193.5, 131.8)
- added REF**: stitch_via, my_SMD:stitch_via0.2mm, F.Cu at (193.5, 132.2)
- added REF**: stitch_via, my_SMD:stitch_via0.2mm, F.Cu at (194.0, 132.2)
- added REF**: stitch_via, my_SMD:stitch_via0.2mm, F.Cu at (193.5, 130.8)
- added REF**: stitch_via, my_SMD:stitch_via0.2mm, F.Cu at (194.5, 131.8)
- added REF**: stitch_via, my_SMD:stitch_via0.2mm, F.Cu at (193.5, 131.2)
- added REF**: stitch_via, my_SMD:stitch_via0.2mm, F.Cu at (194.0, 131.2)
- added REF**: stitch_via, my_SMD:stitch_via0.2mm, F.Cu at (194.0, 131.8)
- added REF**: stitch_via, my_SMD:stitch_via0.2mm, F.Cu at (212.0, 134.2)
- added REF**: stitch_via, my_SMD:stitch_via0.2mm, F.Cu at (212.5, 134.2)
- added REF**: stitch_via, my_SMD:stitch_via0.2mm, F.Cu at (174.6, 119.3)
- added REF**: stitch_via, my_SMD:stitch_via0.2mm, F.Cu at (212.0, 133.8)
- added REF**: stitch_via, my_SMD:stitch_via0.2mm, F.Cu at (212.5, 133.8)
- added REF**: stitch_via, my_SMD:stitch_via0.2mm, F.Cu at (213.5, 134.2)
- added REF**: stitch_via, my_SMD:stitch_via0.2mm, F.Cu at (213.0, 133.8)
- added REF**: stitch_via, my_SMD:stitch_via0.2mm, F.Cu at (213.5, 133.8)
- added REF**: stitch_via, my_SMD:stitch_via0.2mm, F.Cu at (213.0, 134.2)
- added REF**: stitch_via, my_SMD:stitch_via0.2mm, F.Cu at (214.0, 133.8)
- added REF**: stitch_via, my_SMD:stitch_via0.2mm, F.Cu at (214.0, 133.2)
- added REF**: stitch_via, my_SMD:stitch_via0.2mm, F.Cu at (213.5, 133.2)
- added REF**: stitch_via, my_SMD:stitch_via0.2mm, F.Cu at (214.5, 133.8)
- added REF**: stitch_via, my_SMD:stitch_via0.2mm, F.Cu at (171.0, 103.5)
- added REF**: stitch_via, my_SMD:stitch_via0.2mm, F.Cu at (214.5, 134.2)
- added REF**: stitch_via, my_SMD:stitch_via0.2mm, F.Cu at (214.0, 134.2)
- added REF**: stitch_via, my_SMD:stitch_via0.2mm, F.Cu at (213.0, 132.2)
- added REF**: stitch_via, my_SMD:stitch_via0.2mm, F.Cu at (213.0, 132.8)
- added REF**: stitch_via, my_SMD:stitch_via0.2mm, F.Cu at (213.5, 132.2)
- added REF**: stitch_via, my_SMD:stitch_via0.2mm, F.Cu at (213.5, 132.8)
- added REF**: stitch_via, my_SMD:stitch_via0.2mm, F.Cu at (212.0, 133.2)
- added REF**: stitch_via, my_SMD:stitch_via0.2mm, F.Cu at (213.0, 133.2)
- added REF**: stitch_via, my_SMD:stitch_via0.2mm, F.Cu at (212.5, 133.2)
- added REF**: stitch_via, my_SMD:stitch_via0.2mm, F.Cu at (212.5, 132.8)
- added REF**: stitch_via, my_SMD:stitch_via0.2mm, F.Cu at (202.0, 102.0)
- added REF**: stitch_via, my_SMD:stitch_via0.2mm, F.Cu at (212.0, 132.8)
- added REF**: stitch_via, my_SMD:stitch_via0.2mm, F.Cu at (212.0, 132.2)
- added REF**: stitch_via, my_SMD:stitch_via0.2mm, F.Cu at (212.5, 132.2)
- added REF**: stitch_via, my_SMD:stitch_via0.2mm, F.Cu at (213.0, 131.8)
- added REF**: stitch_via, my_SMD:stitch_via0.2mm, F.Cu at (212.5, 131.2)
- added REF**: stitch_via, my_SMD:stitch_via0.2mm, F.Cu at (212.5, 131.8)
- added REF**: stitch_via, my_SMD:stitch_via0.2mm, F.Cu at (212.0, 131.8)
- added REF**: stitch_via, my_SMD:stitch_via0.2mm, F.Cu at (212.0, 130.8)
- added REF**: stitch_via, my_SMD:stitch_via0.2mm, F.Cu at (212.0, 131.2)
- added REF**: MountingHole_3.2mm_M3, Mounting_Holes:MountingHole_3.2mm_M3, F.Cu at (212.0, 140.0)
- added REF**: stitch_via, my_SMD:stitch_via0.2mm, F.Cu at (198.0, 106.0)
- added REF**: stitch_via, my_SMD:stitch_via0.2mm, F.Cu at (193.0, 112.0)
- added REF**: stitch_via, my_SMD:stitch_via0.2mm, F.Cu at (193.0, 108.0)
- added REF**: stitch_via, my_SMD:stitch_via0.2mm, F.Cu at (172.0, 109.0)
- added REF**: stitch_via, my_SMD:stitch_via0.2mm, F.Cu at (167.0, 109.0)
- added REF**: MountingHole_3.2mm_M3, Mounting_Holes:MountingHole_3.2mm_M3, F.Cu at (159.0, 140.0)
- added REF**: stitch_via, my_SMD:stitch_via0.2mm, F.Cu at (157.0, 109.0)
- added REF**: stitch_via, my_SMD:stitch_via0.2mm, F.Cu at (192.7, 103.8)
- added REF**: stitch_via, my_SMD:stitch_via0.2mm, F.Cu at (184.9, 101.2)
- added REF**: stitch_via, my_SMD:stitch_via0.2mm, F.Cu at (176.7, 103.6)
- added REF**: stitch_via, my_SMD:stitch_via0.2mm, F.Cu at (162.0, 98.0)
- added REF**: stitch_via, my_SMD:stitch_via0.2mm, F.Cu at (162.0, 104.0)
- added REF**: stitch_via, my_SMD:stitch_via0.2mm, F.Cu at (157.0, 104.0)
- added REF**: stitch_via, my_SMD:stitch_via0.2mm, F.Cu at (191.9, 119.9)
- added REF**: stitch_via, my_SMD:stitch_via0.2mm, F.Cu at (193.1, 119.3)
- added REF**: stitch_via, my_SMD:stitch_via0.2mm, F.Cu at (191.9, 119.3)
- added REF**: stitch_via, my_SMD:stitch_via0.2mm, F.Cu at (213.0, 103.0)
- added REF**: stitch_via, my_SMD:stitch_via0.2mm, F.Cu at (192.5, 119.3)
- added REF**: stitch_via, my_SMD:stitch_via0.2mm, F.Cu at (193.1, 120.5)
- added REF**: stitch_via, my_SMD:stitch_via0.2mm, F.Cu at (191.9, 120.5)
- added REF**: stitch_via, my_SMD:stitch_via0.2mm, F.Cu at (193.1, 119.9)
- added REF**: stitch_via, my_SMD:stitch_via0.2mm, F.Cu at (192.5, 119.9)
- added REF**: stitch_via, my_SMD:stitch_via0.2mm, F.Cu at (192.5, 120.5)
- added REF**: stitch_via, my_SMD:stitch_via0.2mm, F.Cu at (191.3, 120.5)
- added REF**: stitch_via, my_SMD:stitch_via0.2mm, F.Cu at (191.3, 119.9)
- added REF**: stitch_via, my_SMD:stitch_via0.2mm, F.Cu at (190.7, 119.3)
- added REF**: stitch_via, my_SMD:stitch_via0.2mm, F.Cu at (191.3, 119.3)
- added REF**: stitch_via, my_SMD:stitch_via0.2mm, F.Cu at (208.0, 103.0)
- added REF**: stitch_via, my_SMD:stitch_via0.2mm, F.Cu at (190.7, 119.9)
- added REF**: stitch_via, my_SMD:stitch_via0.2mm, F.Cu at (190.7, 120.5)
- added REF**: stitch_via, my_SMD:stitch_via0.2mm, F.Cu at (174.6, 120.5)
- added REF**: stitch_via, my_SMD:stitch_via0.2mm, F.Cu at (174.0, 120.5)
- added REF**: stitch_via, my_SMD:stitch_via0.2mm, F.Cu at (173.4, 120.5)
- added REF**: stitch_via, my_SMD:stitch_via0.2mm, F.Cu at (172.8, 120.5)
- added REF**: stitch_via, my_SMD:stitch_via0.2mm, F.Cu at (172.2, 120.5)
- added REF**: stitch_via, my_SMD:stitch_via0.2mm, F.Cu at (174.6, 119.9)
- added REF**: stitch_via, my_SMD:stitch_via0.2mm, F.Cu at (174.0, 119.9)
- added REF**: stitch_via, my_SMD:stitch_via0.2mm, F.Cu at (173.4, 119.9)
- added REF**: stitch_via, my_SMD:stitch_via0.2mm, F.Cu at (208.0, 108.0)
- added REF**: stitch_via, my_SMD:stitch_via0.2mm, F.Cu at (172.8, 119.9)
- added REF**: stitch_via, my_SMD:stitch_via0.2mm, F.Cu at (172.2, 119.9)
- added REF**: stitch_via, my_SMD:stitch_via0.2mm, F.Cu at (174.0, 119.3)
- added REF**: stitch_via, my_SMD:stitch_via0.2mm, F.Cu at (173.4, 119.3)
- added REF**: stitch_via, my_SMD:stitch_via0.2mm, F.Cu at (172.8, 119.3)
- added REF**: stitch_via, my_SMD:stitch_via0.2mm, F.Cu at (172.2, 119.3)
- added REF**: stitch_via, my_SMD:stitch_via0.2mm, F.Cu at (175.5, 131.8)
- added REF**: stitch_via, my_SMD:stitch_via0.2mm, F.Cu at (175.0, 131.2)
- added REF**: stitch_via, my_SMD:stitch_via0.2mm, F.Cu at (175.5, 131.2)
- added REF**: stitch_via, my_SMD:stitch_via0.2mm, F.Cu at (175.0, 130.8)
- added REF**: stitch_via, my_SMD:stitch_via0.2mm, F.Cu at (213.0, 108.0)
- added REF**: stitch_via, my_SMD:stitch_via0.2mm, F.Cu at (175.0, 131.8)
- added REF**: stitch_via, my_SMD:stitch_via0.2mm, F.Cu at (175.0, 132.2)
- added REF**: stitch_via, my_SMD:stitch_via0.2mm, F.Cu at (175.5, 132.2)
- added REF**: stitch_via, my_SMD:stitch_via0.2mm, F.Cu at (175.0, 132.8)
- added REF**: stitch_via, my_SMD:stitch_via0.2mm, F.Cu at (175.5, 132.8)
- added REF**: stitch_via, my_SMD:stitch_via0.2mm, F.Cu at (176.0, 131.8)
- added REF**: stitch_via, my_SMD:stitch_via0.2mm, F.Cu at (176.0, 132.2)
- added REF**: stitch_via, my_SMD:stitch_via0.2mm, F.Cu at (176.5, 132.2)
- added REF**: stitch_via, my_SMD:stitch_via0.2mm, F.Cu at (175.0, 134.2)
- added REF**: stitch_via, my_SMD:stitch_via0.2mm, F.Cu at (175.0, 133.2)
- added REF**: stitch_via, my_SMD:stitch_via0.2mm, F.Cu at (213.0, 112.0)
- added REF**: stitch_via, my_SMD:stitch_via0.2mm, F.Cu at (175.5, 133.2)
- added REF**: stitch_via, my_SMD:stitch_via0.2mm, F.Cu at (175.0, 133.8)
- added REF**: stitch_via, my_SMD:stitch_via0.2mm, F.Cu at (175.5, 133.8)
- added REF**: stitch_via, my_SMD:stitch_via0.2mm, F.Cu at (175.5, 134.2)
- added REF**: stitch_via, my_SMD:stitch_via0.2mm, F.Cu at (177.0, 134.2)
- added REF**: stitch_via, my_SMD:stitch_via0.2mm, F.Cu at (177.0, 133.8)
- added REF**: stitch_via, my_SMD:stitch_via0.2mm, F.Cu at (177.5, 133.8)
- added REF**: stitch_via, my_SMD:stitch_via0.2mm, F.Cu at (177.5, 134.2)
- added REF**: stitch_via, my_SMD:stitch_via0.2mm, F.Cu at (176.0, 132.8)
- added REF**: stitch_via, my_SMD:stitch_via0.2mm, F.Cu at (176.5, 132.8)
- added REF**: stitch_via, my_SMD:stitch_via0.2mm, F.Cu at (208.0, 112.0)
- added REF**: stitch_via, my_SMD:stitch_via0.2mm, F.Cu at (176.0, 133.2)
- added REF**: stitch_via, my_SMD:stitch_via0.2mm, F.Cu at (176.5, 133.2)
- added REF**: stitch_via, my_SMD:stitch_via0.2mm, F.Cu at (177.0, 133.2)
- added REF**: stitch_via, my_SMD:stitch_via0.2mm, F.Cu at (176.0, 133.8)
- added REF**: stitch_via, my_SMD:stitch_via0.2mm, F.Cu at (176.5, 133.8)
- added REF**: stitch_via, my_SMD:stitch_via0.2mm, F.Cu at (176.0, 134.2)
- added REF**: stitch_via, my_SMD:stitch_via0.2mm, F.Cu at (176.5, 134.2)
- added REF**: stitch_via, my_SMD:stitch_via0.2mm, F.Cu at (194.0, 133.2)
- added REF**: stitch_via, my_SMD:stitch_via0.2mm, F.Cu at (193.5, 133.2)
- added REF**: stitch_via, my_SMD:stitch_via0.2mm, F.Cu at (194.0, 132.8)
- added REF**: stitch_via, my_SMD:stitch_via0.2mm, F.Cu at (198.0, 112.0)
- added REF**: stitch_via, my_SMD:stitch_via0.2mm, F.Cu at (193.5, 132.8)
- added REF**: stitch_via, my_SMD:stitch_via0.2mm, F.Cu at (194.5, 133.2)
- added REF**: stitch_via, my_SMD:stitch_via0.2mm, F.Cu at (195.0, 133.2)
- added REF**: stitch_via, my_SMD:stitch_via0.2mm, F.Cu at (194.5, 132.8)
- added REF**: stitch_via, my_SMD:stitch_via0.2mm, F.Cu at (195.0, 132.8)
- added REF**: stitch_via, my_SMD:stitch_via0.2mm, F.Cu at (195.0, 132.2)
- added REF**: stitch_via, my_SMD:stitch_via0.2mm, F.Cu at (195.5, 133.2)
- added REF**: stitch_via, my_SMD:stitch_via0.2mm, F.Cu at (194.5, 132.2)
- added REF**: stitch_via, my_SMD:stitch_via0.2mm, F.Cu at (194.0, 134.2)
- added REF**: stitch_via, my_SMD:stitch_via0.2mm, F.Cu at (194.0, 133.8)
- C1: value C -> 0.022uF; footprint Capacitors_SMD:C_0603 -> Resistors_SMD:R_0402
- C10, C11, C7, C8, C9: value C -> 0.1uF; footprint Capacitors_SMD:C_0603 -> Resistors_SMD:R_0402; moved to B.Cu
- C12, C13: footprint Capacitors_SMD:C_0603 -> Resistors_SMD:R_0402
- C2, C3: value C -> 1uF
- C4: value C -> 2.2uF; footprint Capacitors_SMD:C_0603 -> Resistors_SMD:R_0402
- C5: value C -> 4.7uF
- C6: value C -> 0.1uF; footprint Capacitors_SMD:C_0603 -> Resistors_SMD:R_0402
- J2: value Conn_01x09 -> Conn_01x19; footprint Pin_Headers:Pin_Header_Straight_1x09_Pitch2.54mm -> Pin_Headers:Pin_Header_Straight_1x19_Pitch2.54mm
- Q1, Q10, Q11, Q12, Q2, Q3, Q4, Q5, Q6, Q7, Q8, Q9: footprint TO_SOT_Packages_SMD:TO-252-3_TabPin2 -> my_SMD:PQFN8_5x6
- R1: value R -> 0R; footprint Resistors_SMD:R_0603 -> Resistors_SMD:R_0402
- R10, R11: value R -> 56R; footprint Resistors_SMD:R_0603 -> Resistors_SMD:R_0402
- R2, R3, R5, R6, R8, R9: value R -> 10R
- R4, R7: value R -> 0.01R; footprint Resistors_SMD:R_0603 -> Resistors_SMD:R_2010
- moved J2 49.3 mm to (207.0, 96.3), turned to 270 degrees
- moved J1 37.9 mm to (160.0, 115.0), turned to 90 degrees
- moved R4 37.8 mm to (195.0, 122.0), turned to 90 degrees
- moved R2 31.9 mm to (206.4, 122.2), turned to 270 degrees
- moved C10 29.7 mm to (180.7, 117.0)
- moved R9 28.8 mm to (161.9, 122.2), turned to 270 degrees
- moved C11 25.6 mm to (178.8, 117.0)
- moved R3 23.8 mm to (198.9, 122.2), turned to 270 degrees
- moved R8 23.6 mm to (169.4, 122.2), turned to 270 degrees
- moved R7 21.8 mm to (176.5, 122.0), turned to 90 degrees
- moved Q1 16.1 mm to (208.0, 132.0), turned to 270 degrees
- moved C12 16.0 mm to (170.9, 105.0)
- moved C13 15.8 mm to (167.0, 105.0)
- moved R10 15.7 mm to (168.3, 105.0)
- moved R11 15.5 mm to (169.6, 105.0)
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Connections:
- J2 pad 1: /AH -> +3V3
- J2 pad 2: /AL -> GND
- J2 pad 3: /BH -> /nOCTW
- J2 pad 4: /BL -> /nFAULT
- J2 pad 5: /CH -> /nCS
- J2 pad 6: /CL -> /SDI
- J2 pad 7: /REF -> /SDO
- J2 pad 8: /SO1 -> /SCLK
- J2 pad 9: /SO2 -> /DC_CAL
- U1 pad 45: Net-(U1-Pad45) -> +3V3
Routing:
- net GND: track 0.00 -> 60.7 mm, vias 0 -> 6
- net /SL_A: track 0.00 -> 40.8 mm, vias 0 -> 2
- net +3V3: track 0.00 -> 34.6 mm
- net /SL_B: track 0.00 -> 25.7 mm, vias 0 -> 2
- net /GL_C: track 0.00 -> 24.6 mm
- net /SH_A: track 0.00 -> 23.7 mm, vias 0 -> 1
- net /SH_C: track 0.00 -> 23.5 mm, vias 0 -> 1
- net /GH_A: track 0.00 -> 23.5 mm
- net /REF: track 0.00 -> 19.6 mm
- net /GH_C: track 0.00 -> 19.0 mm
- net /GL_A: track 0.00 -> 18.7 mm
- net /CL: track 0.00 -> 18.7 mm
- net /nOCTW: track 0.00 -> 17.1 mm
- net /CH: track 0.00 -> 16.6 mm
- net /nFAULT: track 0.00 -> 15.6 mm
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- added copper zone on F.Cu, net /SH_A
- added copper zone on F.Cu, net /SH_B
- added copper zone on F.Cu, net /SH_C
- added copper zone on F.Cu, net /SL_A
- added copper zone on F.Cu, net /SL_B
- added copper zone on B.Cu, net GND
- added copper zone on F.Cu, net GND
- added copper zone on B.Cu, net VBUS
- added copper zone on F.Cu, net VBUS
Other:
- board outline added: 61 x 49 mm
- net class Default: clearance 0.2 -> 0.127; trace_width 0.25 -> 0.127; via_dia 0.6 -> 0.5; via_drill 0.4 -> 0.3
- net class Fet_drive added: clearance 0.127, trace_width 0.3, via_dia 0.5, via_drill 0.3
- net class logic_v added: clearance 0.127, trace_width 0.2, via_dia 0.4, via_drill 0.3
- rule trace_clearance: 0.2 -> 0.127
- rule trace_min: 0.2 -> 0.127
- rule via_min_drill: 0.3 -> 0.2
- rule via_min_size: 0.4 -> 0.3
- board text added: "3v3"
- board text added: "AH"
- board text added: "AL"
- board text added: "BH"
- board text added: "BL"
- board text added: "BLDC driver REV A Jon Anderson April 2018 jonnyando@gmail.com"
- board text added: "CAL"
- board text added: "CH"
- board text added: "CL"
- board text added: "CLK"
- board text added: "EN"
- board text added: "GND"
- board text added: "PWR"
- board text added: "REF"
- board text added: "SDI"
- board text added: "SDO"
- board text added: "SO1"
- board text added: "SO2"
- board text added: "TODO:"
- board text added: "nCS"
- board text added: "nFAULT"
- board text added: "nOCTW"
- board text removed: "V+ can go straight to the back plane Come up through via stitching to the FETs SH pads can stitch down to power resistors for shunts, and then connect back to the GND plane somehow"
