File: motor_driver/motor_driver.sch (KiCad schematic (older format))
At the start: 41 parts, among them J1 Power_in, J2 Conn_01x09, J3 Conn_01x10, J4 Screw_Terminal_01x03, Q1 N_MOSFET, Q10 N_MOSFET, Q11 N_MOSFET, Q12 N_MOSFET, Q2 N_MOSFET, Q3 N_MOSFET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

Commit message: Finished layout and generated gerbers
Parts:
- removed J2: Conn_01x09, Pin_Headers:Pin_Header_Straight_1x09_Pitch2.54mm, symbol Conn_01x09
- removed J3: Conn_01x10, Pin_Headers:Pin_Header_Straight_1x10_Pitch2.54mm, symbol Conn_01x10
- added C14: CP1, Capacitors_SMD:CP_Elec_6.3x7.7, symbol CP1
- added D1: LED, LEDs:LED_0805, symbol LED
- added J2: Conn_01x19, Pin_Headers:Pin_Header_Straight_1x19_Pitch2.54mm, symbol Conn_01x19
- added R12: 1KR, Resistors_SMD:R_0805, symbol R
- C1: value C -> 0.022uF; footprint Capacitors_SMD:C_0603 -> Resistors_SMD:R_0402
- C10, C11, C6, C7, C8, C9: value C -> 0.1uF; footprint Capacitors_SMD:C_0603 -> Resistors_SMD:R_0402
- C12, C13: footprint Capacitors_SMD:C_0603 -> Resistors_SMD:R_0402
- C2, C3: value C -> 1uF
- C4: value C -> 2.2uF; footprint Capacitors_SMD:C_0603 -> Resistors_SMD:R_0402
- C5: value C -> 4.7uF
- Q1, Q10, Q11, Q12, Q2, Q3, Q4, Q5, Q6, Q7, Q8, Q9: footprint TO_SOT_Packages_SMD:TO-252-3_TabPin2 -> my_SMD:PQFN8_5x6
- R1: value R -> 0R; footprint Resistors_SMD:R_0603 -> Resistors_SMD:R_0402
- R10, R11: value R -> 56R; footprint Resistors_SMD:R_0603 -> Resistors_SMD:R_0402
- R2, R3, R5, R6, R8, R9: value R -> 10R
- R4, R7: value R -> 0.01R; footprint Resistors_SMD:R_0603 -> Resistors_SMD:R_2010
Connections:
- net +3V3: now also U1.45 (VDD_SPI), J2.1 (Pin_1), R12.2
- net AH: now also J2.11 (Pin_11)
- net AL: now also J2.12 (Pin_12)
- net BH: now also J2.13 (Pin_13)
- net BL: now also J2.14 (Pin_14)
- net CH: now also J2.15 (Pin_15)
- net CL: now also J2.16 (Pin_16)
- net DC_CAL: now also J2.9 (Pin_9)
- net EN_GATE: now also J2.10 (Pin_10)
- net GND: now also C14.2, D1.1 (K), J2.2 (Pin_2)
- net REF: now also J2.17 (Pin_17)
- net SCLK: now also J2.8 (Pin_8)
- net SDI: now also J2.6 (Pin_6)
- net SDO: now also J2.7 (Pin_7)
- net SO1: now also J2.18 (Pin_18)
- net SO2: now also J2.19 (Pin_19)
- net VBUS: now also C14.1
- net nCS: now also J2.5 (Pin_5)
- net nFAULT: now also J2.4 (Pin_4)
- net nOCTW: now also J2.3 (Pin_3)
- new net: D1.2 (A), R12.1
